File: PCB/Probe/probe_v2-0/probe.kicad_pcb (KiCad board)
At the start: 4 copper layers, 50 x 50 mm, 72 parts, among them J1 PWR, J2 USB_B_Micro, J3 TP, J4 Temp_Screw, J6 Inter Board, J7 Au1, J8 Au2, SW1 SW_En, SW2 SW_Boot, U1 MCP4725xxx-xCH, U10 4xSwitch, U12 SP3485EN, U13 LPS28DFW, U2 AMS1117-3.3, U3 AMS1117-5.0, U4 ESP32-S2-MINI-1, U5 LM358, U6 4xSwitch, U7 4xSwitch, U8 4xSwitch, U9 LM358

Commit message: All PCBs Done
Parts:
- added J5: Data, Connector_PinHeader_2.54mm:PinHeader_1x02_P2.54mm_Vertical, F.Cu at (143.4, 47.0)
Routing:
- net D-: track 22.8 -> 77.5 mm
- net D+: track 25.7 -> 70.3 mm
- added copper zone on B.Cu, net GND
Other:
- board text added: "D+ D-"
