File: PCB/Probe/probe_v2-0/probe.kicad_sch (KiCad schematic)
At the start: 79 parts, among them J1 PWR, J10 Au4, J2 USB_B_Micro, J3 TP, J4 Temp_Screw, J6 Inter Board, J7 Au1, J8 Au2, J9 Au3, SW1 SW_En, SW2 SW_Boot, U1 MCP4725xxx-xCH, U10 4xSwitch, U11 4xSwitch, U12 SP3485EN, U13 LPS28DFW, U2 AMS1117-3.3, U3 AMS1117-5.0, U4 ESP32-S2-MINI-1, U5 LM358, U6 4xSwitch, U7 4xSwitch, U8 4xSwitch, U9 LM358

Commit message: Created PCB and New Schematic Version
Parts:
- removed J10: Au4, symbol Connector:Conn_01x02_Socket
- removed J9: Au3, symbol Connector:Conn_01x02_Socket
- removed U11: 4xSwitch, Package_SO:TSSOP-14_4.4x5mm_P0.65mm, symbol ThesisLibrary:TS3A4751PWR
- D4: footprint (none) -> LED_SMD:LED_0603_1608Metric; now fitted; now in the parts list
- J4: footprint TerminalBlock_Phoenix:TerminalBlock_Phoenix_MKDS-1,5-3_1x03_P5.00mm_Horizontal -> ThesisLib:3-Wire Solder Pads; symbol Connector:Screw_Terminal_01x03 -> Connector:Conn_01x03_Socket
- J7, J8: footprint (none) -> ThesisLib:Au_Electrode
- R5: value 10K -> 1K; footprint (none) -> Resistor_SMD:R_0603_1608Metric; now fitted; now in the parts list
- U13: footprint LPS28DFW:CCLGA-7L -> ThesisLib:CCLGA-7L
Connections:
- net AMP: no longer U7.10 (COM4), U7.9 (COM3)
- net GND: now also U7.10 (COM4), U7.9 (COM3); no longer C15.2, C16.2, C17.2, C18.2
- net at U7.11 (NO4): now also J8.2 (Pin_2), U7.3 (NO2); no longer U8.10 (COM4)
- net at J7.1 (Pin_1), U7.1 (NO1): now also U7.8 (NO3); no longer U8.2 (COM1)
- net C_AMP: now reaches U8.9 (COM3)
- net C_AMP: now also C17.2; no longer U7.8 (NO3)
- net Au+1 Shield renamed Au+ Shield
- net Au-1 Shield renamed Au- Shield
- net SW_Au+1 renamed SW_Au+
- net SW_Au+1_GND renamed SW_UBD
- net SW_Au+1_SH+ renamed SW_Au+_SH+
- net SW_Au+1_SH- renamed SW_Au+_SH-
- net SW_Au+2 renamed SW_Au+_GND
- net SW_Au+2_GND renamed SW_AMP
- net SW_Au+2_SH+: no longer names the net of U4.33 (GPIO37)
- net SW_Au+2_SH-: no longer names the net of U4.41 (GPIO45)
- net SW_Au-1 renamed SW_Au-
- net SW_Au-1_GND renamed SW_DAC
- net SW_Au-1_SH+ renamed SW_Au-_SH+
- net SW_Au-1_SH- renamed SW_Au-_SH-
- net SW_Au-2 renamed SW_Au-_GND
- net SW_Au-2_GND renamed SW_SGN
- net SW_Au-2_SH+: no longer names the net of U4.34 (GPIO38)
- net SW_Au-2_SH-: no longer names the net of U4.26 (SPI_CS1/GPIO26)
- new net C_DAC: C16.2, U8.4 (COM2)
- new net C_SGN: C18.2, U8.10 (COM4)
- new net C_UBD: C15.2, U8.2 (COM1)
- no-connect marks 4 -> 8
Other:
- note added: "SW Cap"
- note added: "SW GRD"
- note added: "SW Guard"
- note added: "Switch R2-GND"
- note added: "To ground <-------"
- note removed: "SW GRD Au1"
- note removed: "SW GRD Au2"
- note removed: "SW Guard (Au1)"
- note removed: "SW Guard (Au2)"
- note removed: "Switch "R2""
- note removed: "Switch GND"
- moved on the sheet: C15, C16, C17, C18, J7, J8, R24, R25, R26, U10, U4, U7

Commit message: All PCBs Done
Parts:
- added J5: Data, Connector_PinHeader_2.54mm:PinHeader_1x02_P2.54mm_Vertical, symbol Connector_Generic:Conn_01x02
- C1, C13, C14, C15, C16, C17, C18, C19, C20, C21, C22, C23, C3, C5, C8: Cost (none) -> 0.011; JLC Part no. (none) -> C1525
- C10, C2, C4, C6, C7, C9: Cost (none) -> 0.0443; JLC Part no. (none) -> C12891
- C11, C12: Cost (none) -> 0.0056; JLC Part no. (none) -> C19702
- D1: Cost (none) -> 0.0276; JLC Part no. (none) -> C8678
- D4: Cost (none) -> 0.0056; JLC Part no. (none) -> C2286
- J1, J3, J6, J7, J8: now not fitted
- J2: Cost (none) -> 0.0368; Extended (none) -> Yes; JLC Part no. (none) -> C404969
- J4: value Temp_Screw -> Temp_Pads; now not fitted
- R10, R8, R9: Cost (none) -> 0.0011; JLC Part no. (none) -> C23025
- R11, R12, R13: Cost (none) -> 0.0010; JLC Part no. (none) -> C4211
- R14, R15, R16: Cost (none) -> 0.0010; JLC Part no. (none) -> C22984
- R17, R18, R19, R20: Cost (none) -> 0.0011; JLC Part no. (none) -> C22950
- R21, R5: Cost (none) -> 0.0010; JLC Part no. (none) -> C21190
- R22, R6, R7: Cost (none) -> 0.0009; JLC Part no. (none) -> C25804
- R23: Cost (none) -> 0.0011; JLC Part no. (none) -> C22787
- R24, R25, R26, R27, R28: Cost (none) -> 0.0011; JLC Part no. (none) -> C23162
- SW1, SW2: Cost (none) -> 0.0423; JLC Part no. (none) -> C720477
- U1: Cost (none) -> 0.9; Extended (none) -> Yes; JLC Part no. (none) -> C144198
- U10, U6, U7, U8: Cost (none) -> 1.0695; Extended (none) -> Yes
- U12: Cost (none) -> 0.2048; JLC Part no. (none) -> C8963
- U13: Cost (none) -> 3.792; Extended (none) -> Yes; JLC Part no. (none) -> C3263277
- U2: Cost (none) -> 0.1653; JLC Part no. (none) -> C6186
- U3: Cost (none) -> 0.1913; JLC Part no. (none) -> C6187
- U4: Cost (none) -> 1.8960; Extended (none) -> Yes; JLC Part no. (none) -> C3013906
- U5, U9: Cost (none) -> 0.0758; JLC Part no. (none) -> C7950
Connections:
- net D+: now also J5.1 (Pin_1)
- net D-: now also J5.2 (Pin_2)
